File: Capteur_KICAD/Capteur_KICAD.kicad_sch (KiCad schematic)
At the start: 20 parts, among them J1 Power, J2 Digital/PWM, J3 Analog, J4 Digital/PWM

Commit message: Updating PCB, proposition of final PCB
Parts:
- added C5: 100n, Capacitor_THT:C_Disc_D4.3mm_W1.9mm_P5.00mm, symbol Device:C
- added R7: 1k, Resistor_THT:R_Axial_DIN0204_L3.6mm_D1.6mm_P5.08mm_Horizontal, symbol Device:R
- C1, C2, C3: footprint Capacitor_THT:CP_Axial_L10.0mm_D4.5mm_P15.00mm_Horizontal -> Capacitor_THT:C_Disc_D4.3mm_W1.9mm_P5.00mm
- C4: footprint Capacitor_THT:CP_Axial_L10.0mm_D4.5mm_P15.00mm_Horizontal -> Capacitor_THT:C_Rect_L7.0mm_W4.5mm_P5.00mm
- R1, R3: footprint Resistor_THT:R_Axial_DIN0204_L3.6mm_D1.6mm_P2.54mm_Vertical -> Resistor_THT:R_Axial_DIN0204_L3.6mm_D1.6mm_P5.08mm_Horizontal
- R6: footprint Resistor_THT:R_Axial_DIN0204_L3.6mm_D1.6mm_P2.54mm_Vertical -> Resistor_THT:R_Axial_DIN0207_L6.3mm_D2.5mm_P7.62mm_Horizontal
- U4: footprint Package_DIP:CERDIP-8_W7.62mm_SideBrazed_LongPads -> LTC1050ACN8_PBF:PDIP-8_N
Connections:
- net +5V: now also R7.2; no longer U2.1 (V+)
- net 2: now also C5.1
- net 3: now also U7.2 (DT); no longer U7.3 (SW)
- net 4: now also U7.3 (SW); no longer U7.2 (DT)
- net A2: now also U2.2 (V-)
- net A3: no longer U2.2 (V-)
- net GND: now also C5.2
- net at R3.1, U4.2 (-IN), U6.7 (P0B): now also C4.1; no longer C4.2
- net at R6.1, U4.6 (OUT): now also C4.2, R3.2
- net at C3.2, U4.7 (V+): no longer C4.1, R3.2
- new net: R7.1, U2.1 (V+)
Other:
- moved on the sheet: C4, U1, U2, U5, U7, U8

Commit message: Updating PCB on KiCad, final proposition without 3D model
Parts:
- removed C3: 100n, Capacitor_THT:C_Disc_D4.3mm_W1.9mm_P5.00mm, symbol Device:C
- R5: footprint Resistor_THT:R_Axial_DIN0204_L3.6mm_D1.6mm_P2.54mm_Vertical -> Resistor_THT:R_Axial_DIN0204_L3.6mm_D1.6mm_P5.08mm_Horizontal
Connections:
- net +5V: now also U4.7 (V+), U6.8 (Vdd)
- net 10: now also U6.1 (CS); no longer U6.4 (Vss)
- net A2: now also R7.1, U2.1 (V+); no longer U2.2 (V-)
- net GND: now also U2.2 (V-), U4.4 (V-), U6.4 (Vss)
- no-connect marks 5 -> 3

Commit message: Pin shape correction
Parts:
- U4: footprint LTC1050ACN8_PBF:PDIP-8_N -> Package_DIP:CERDIP-8_W7.62mm_SideBrazed_LongPads_Socket
Changed lines of the file:
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@@
 			)
 		)
-		(property "Footprint" "LTC1050ACN8_PBF:PDIP-8_N"
+		(property "Footprint" "Package_DIP:CERDIP-8_W7.62mm_SideBrazed_LongPads_Socket"
 			(at 96.52 135.89 0)
 			(effects
